Commit message: created a basic urdf

File: rover_ws/src/rover_description/urdf/rover.urdf (robot description, URDF)
Before this commit: robot rover, 1 links, 0 joints
Links:
- added link wheel_front_left; visual cylinder length=0.1 radius=0.1
- added link wheel_front_right; visual cylinder length=0.1 radius=0.1
- added link wheel_mid_left; visual cylinder length=0.1 radius=0.1
- added link wheel_mid_right; visual cylinder length=0.1 radius=0.1
- added link wheel_rear_left; visual cylinder length=0.1 radius=0.1
- added link wheel_rear_right; visual cylinder length=0.1 radius=0.1
- link base_link: geometry visual box size=0.7 0.45 0.2
Joints:
- added joint joint_wheel_front_left: type continuous, parent base_link, child wheel_front_left, origin xyz=0.25 0.275 -0.1 rpy=0 0 0, axis 0 1 0
- added joint joint_wheel_front_right: type continuous, parent base_link, child wheel_front_right, origin xyz=0.25 -0.275 -0.1 rpy=0 0 0, axis 0 1 0
- added joint joint_wheel_mid_left: type continuous, parent base_link, child wheel_mid_left, origin xyz=0.0 0.275 -0.1 rpy=0 0 0, axis 0 1 0
- added joint joint_wheel_mid_right: type continuous, parent base_link, child wheel_mid_right, origin xyz=0.0 -0.275 -0.1 rpy=0 0 0, axis 0 1 0
- added joint joint_wheel_rear_left: type continuous, parent base_link, child wheel_rear_left, origin xyz=-0.25 0.275 -0.1 rpy=0 0 0, axis 0 1 0
- added joint joint_wheel_rear_right: type continuous, parent base_link, child wheel_rear_right, origin xyz=-0.25 -0.275 -0.1 rpy=0 0 0, axis 0 1 0
