Commit message: new changes to motor speeds and urdf

File: rover_ws/src/motor_node/urdf/arm.urdf (robot description, URDF)
Before this commit: robot robot_arm, 5 links, 4 joints
Links:
- added link pitch; visual box size=0.05 0.05 0.05
- added link roll; visual box size=0.05 0.05 0.05
- added link yaw; visual box size=0.05 0.05 0.05
- link ee_link: geometry visual box size=0.1 0.1 0.15
Joints:
- added joint pitch_joint: type revolute, parent yaw, child pitch, origin xyz=-0.05 -0.05 0 rpy=0 0 0, axis 1 0 0, limit lower=-0.0873 upper=4.7997 effort=100 velocity=1.0
- added joint roll_joint: type revolute, parent pitch, child roll, origin xyz=0 0 0.075 rpy=0 0 0, axis 0 0 1, limit lower=-3.2288 upper=3.2288 effort=100 velocity=1.0
- added joint yaw_joint: type revolute, parent arm2, child yaw, origin xyz=0 -0.05 0.6 rpy=0 0 0, axis 0 1 0, limit lower=-1.6581 upper=3.2288 effort=100 velocity=1.0
- joint base_joint: limit lower=-3.14 upper=3.14 effort=100 velocity=1.0 -> lower=-3.2288 upper=3.2288 effort=100 velocity=1.0
- joint ee_joint: origin xyz=0 0 0.5 rpy=0 0 0 -> xyz=0 0 0.05 rpy=0 0 0; parent arm2 -> roll
- joint elbow_joint: limit lower=0 upper=4.71 effort=100 velocity=1.0 -> lower=-0.0873 upper=4.7997 effort=100 velocity=1.0
- joint shoulder_joint: limit lower=0 upper=3.14 effort=100 velocity=1.0 -> lower=-0.0873 upper=3.2288 effort=100 velocity=1.0
